Commit message: chore(release): SOTA Paper V1.0 Prep - SafeVLA: Language-Conditioned CBFs

File: fleet_trinity_dashboard/public/robots/fastbot/fastbot.urdf (robot description, URDF)
Before this commit: robot fastbot, 9 links, 8 joints
Links:
- removed link fl_wheel
- removed link fr_wheel
- removed link rl_wheel
- removed link rr_wheel
- added link front_stand; visual sphere radius=0.12
- added link l_wheel; visual cylinder length=0.08 radius=0.12
- added link r_wheel; visual cylinder length=0.08 radius=0.12
Joints:
- removed joint fl_wheel_joint
- removed joint fr_wheel_joint
- removed joint rl_wheel_joint
- removed joint rr_wheel_joint
- added joint front_stand_joint: type fixed, parent base_link, child front_stand, origin xyz=0.25 0 0.12 rpy=0 0 0
- added joint l_wheel_joint: type continuous, parent base_link, child l_wheel, origin xyz=-0.25 0.29 0.12 rpy=0 0 0, axis 0 1 0
- added joint r_wheel_joint: type continuous, parent base_link, child r_wheel, origin xyz=-0.25 -0.29 0.12 rpy=0 0 0, axis 0 1 0
